File: schematics/drone-beacon/drone-beacon.kicad_sch (KiCad schematic)
At the start: 13 parts, among them J1 ESP32 Flashing connector, J2 Power Input, SW1 Model selection, U1 ESP32-WROOM-32U, U2 AMS1117-3.3, U3 L80-R

Commit message: Update schematics
Signed-off-by: LAMBS Pierre-Antoine <pierreantoine.lambs@gmail.com>
Parts:
- J2: footprint (none) -> Connector_PinHeader_2.00mm:PinHeader_1x02_P2.00mm_Vertical
- U2: footprint Package_TO_SOT_SMD:SOT-89-3 -> Package_TO_SOT_SMD:SOT-223
Changed lines of the file:
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@@
 			)
 		)
-		(property "Footprint" "Package_TO_SOT_SMD:SOT-89-3"
+		(property "Footprint" "Package_TO_SOT_SMD:SOT-223"
 			(at 148.59 20.32 0)
 			(effects
@@
 			)
 		)
-		(property "Footprint" ""
+		(property "Footprint" "Connector_PinHeader_2.00mm:PinHeader_1x02_P2.00mm_Vertical"
 			(at 96.52 30.48 0)
 			(effects

Commit message: Update schematics
Signed-off-by: LAMBS Pierre-Antoine <pierreantoine.lambs@gmail.com>
Parts:
- C1, C2, C3, C4: footprint Capacitor_SMD:C_0201_0603Metric -> Capacitor_SMD:C_0402_1005Metric_Pad0.74x0.62mm_HandSolder
- D1: footprint LED_SMD:LED_0201_0603Metric -> LED_SMD:LED_0402_1005Metric_Pad0.77x0.64mm_HandSolder
- R1, R3: footprint Resistor_SMD:R_0201_0603Metric -> Resistor_SMD:R_0402_1005Metric_Pad0.72x0.64mm_HandSolder
- U3: value L80-R -> L96; footprint RF_GPS:Quectel_L96 -> QUECTEL_L96:L96; symbol RF_GPS:L80-R -> L96:L96-M33; Manufacturer_Name (none) -> Quectel; Manufacturer_Part_Number (none) -> L96-M33; Mouser Part Number (none) -> 277-L96-M33; Mouser Price/Stock (none) -> https://www.mouser.co.uk/ProductDetail/Quectel/L96-M33?qs=G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
Connections:
- net +3.3V: now also U3.23 (RESET), U3.9 (VDD); no longer U3.4 (VCC)
- net GND: now also U3.10 (GND3), U3.11 (GND4), U3.13 (GND6), U3.14 (GND7), U3.15 (GND8), U3.18 (GND9), U3.19 (GND10), U3.21 (GND11), U3.22 (GND12), U3.27 (GND13), U3.31 (GND14), U3.4 (GND1), U3.5 (GND2); no longer U3.3 (GND)
- net GPS_PPS: now also U3.29 (TIMEPULSE); no longer U3.6 (1PPS)
- net GPS_RX: now also U3.26 (RXD1); no longer U3.1 (RXD1)
- net GPS_TX: now also U3.25 (TXD1); no longer U3.2 (TXD1)
- no-connect marks 26 -> 33
Other:
- moved on the sheet: SW1

Commit message: Update schematics (WIP)
Signed-off-by: LAMBS Pierre-Antoine <pierreantoine.lambs@gmail.com>
Parts:
- added R2: 0, symbol Device:R
Connections:
- net +3.3V: now also U3.8 (V_BCKP)
- net DIP1: now also U1.16 (IO13); no longer U1.14 (IO12)
- net RF_OUT: now reaches U3.16 (RF_OUT)
- net RF_OUT: now also R2.2
- net RF_IN: now reaches U3.17 (RF_IN)
- net RF_IN: now also R2.1
- no-connect marks 33 -> 30
Changed lines of the file:
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@@
-	)
-	(junction
-		(at 93.98 91.44)
-		(diameter 0)
-		(color 0 0 0 0)
 	)
 	(junction
@@
 		(color 0 0 0 0)
 	)
+	(junction
+		(at 96.52 76.2)
+		(diameter 0)
+		(color 0 0 0 0)
+	)
 	(no_connect
 		(at 67.31 57.15)
@@
 	)
 	(no_connect
-		(at 134.62 55.88)
-	)
-	(no_connect
-		(at 96.52 73.66)
+		(at 67.31 49.53)
 	)
 	(no_connect
@@
 	)
 	(no_connect
-		(at 67.31 52.07)
-	)
-	(no_connect
 		(at 36.83 77.47)
 	)
@@
 	)
 	(no_connect
-		(at 96.52 93.98)
-	)
-	(no_connect
 		(at 134.62 73.66)
 	)
@@
 	(wire
 		(pts
+			(xy 93.98 81.28) (xy 88.9 81.28)
+		)
+		(stroke
+			(width 0)
+			(type default)
+		)
+	)
+	(wire
+		(pts
 			(xy 135.89 91.44) (xy 134.62 91.44)
 		)
@@
 	(wire
 		(pts
-			(xy 93.98 91.44) (xy 93.98 95.25)
+			(xy 161.29 99.06) (xy 163.83 99.06)
+		)
+		(stroke
+			(width 0)
+			(type default)
+		)
+	)
+	(wire
+		(pts
+			(xy 151.13 99.06) (xy 153.67 99.06)
+		)
+		(stroke
+			(width 0)
+			(type default)
+		)
+	)
+	(wire
+		(pts
+			(xy 134.62 55.88) (xy 138.43 55.88)
 		)
 		(stroke
@@
 	(wire
 		(pts
+			(xy 88.9 81.28) (xy 88.9 82.55)
+		)
+		(stroke
+			(width 0)
+			(type default)
+		)
+	)
+	(wire
+		(pts
 			(xy 135.89 81.28) (xy 134.62 81.28)
 		)
@@
 	(wire
 		(pts
+			(xy 96.52 73.66) (xy 96.52 76.2)
+		)
+		(stroke
+			(width 0)
+			(type default)
+		)
+	)
+	(wire
+		(pts
 			(xy 93.98 86.36) (xy 93.98 88.9)
 		)
@@
 	(wire
 		(pts
-			(xy 67.31 49.53) (xy 76.2 49.53)
-		)
-		(stroke
-			(width 0)
-			(type default)
-		)
-	)
-	(wire
-		(pts
 			(xy 93.98 66.04) (xy 93.98 78.74)
 		)
@@
 	(wire
 		(pts
+			(xy 90.17 93.98) (xy 96.52 93.98)
+		)
+		(stroke
+			(width 0)
+			(type default)
+		)
+	)
+	(wire
+		(pts
 			(xy 158.75 78.74) (xy 165.1 78.74)
 		)
@@
 		(pts
 			(xy 93.98 83.82) (xy 93.98 86.36)
+		)
+		(stroke
+			(width 0)
+			(type default)
+		)
+	)
+	(wire
+		(pts
+			(xy 67.31 52.07) (xy 76.2 52.07)
 		)
 		(stroke
@@
 		)
 	)
+	(label "RF_OUT"
+		(at 90.17 93.98 180)
+		(effects
+			(font
+				(size 1.27 1.27)
+			)
+			(justify right bottom)
+		)
+	)
 	(label "ESP32_BOOT"
 		(at 171.45 54.61 180)
@@
 		)
 	)
+	(label "RF_OUT"
+		(at 163.83 99.06 0)
+		(effects
+			(font
+				(size 1.27 1.27)
+			)
+			(justify left bottom)
+		)
+	)
 	(label "GPS_RX"
 		(at 76.2 62.23 0)
@@
 		)
 	)
+	(label "RF_IN"
+		(at 151.13 99.06 180)
+		(effects
+			(font
+				(size 1.27 1.27)
+			)
+			(justify right bottom)
+		)
+	)
 	(label "DIP1"
-		(at 76.2 49.53 0)
+		(at 76.2 52.07 0)
 		(effects
 			(font
@@
 			)
 			(justify right bottom)
+		)
+	)
+	(label "RF_IN"
+		(at 138.43 55.88 0)
+		(effects
+			(font
+				(size 1.27 1.27)
+			)
+			(justify left bottom)
 		)
 	)
@@
 	(symbol
 		(lib_id "power:GND")
-		(at 93.98 95.25 0)
+		(at 88.9 82.55 0)
 		(unit 1)
 		(exclude_from_sim no)
@@
 		(fields_autoplaced yes)
 		(property "Reference" "#PWR010"
-			(at 93.98 101.6 0)
+			(at 88.9 88.9 0)
 			(effects
 				(font
@@
 		)
 		(property "Value" "GND"
-			(at 93.98 100.33 0)
+			(at 88.9 87.63 0)
 			(effects
 				(font
@@
 		)
 		(property "Footprint" ""
-			(at 93.98 95.25 0)
+			(at 88.9 82.55 0)
 			(effects
 				(font
@@
 		)
 		(property "Datasheet" ""
-			(at 93.98 95.25 0)
+			(at 88.9 82.55 0)
 			(effects
 				(font
@@
 		)
 		(property "Description" "Power symbol creates a global label with name \"GND\" , ground"
-			(at 93.98 95.25 0)
+			(at 88.9 82.55 0)
 			(effects
 				(font
@@
 					(unit 1)
 				)
+			)
+		)
+	)
+	(symbol
+		(lib_id "Device:R")
+		(at 157.48 99.06 90)
+		(unit 1)
+		(exclude_from_sim no)
+		(in_bom yes)
+		(on_board yes)
+		(dnp no)
+		(fields_autoplaced yes)
+		(property "Reference" "R2"
+			(at 157.48 92.71 90)
+			(effects
+				(font
+					(size 1.27 1.27)
+				)
+			)
+		)
+		(property "Value" "0"
+			(at 157.48 95.25 90)
+			(effects
+				(font
+					(size 1.27 1.27)
+				)
+			)
+		)
+		(property "Footprint" ""
+			(at 157.48 100.838 90)
+			(effects
+				(font
+					(size 1.27 1.27)
+				)
+				(hide yes)
+			)
+		)
+		(property "Datasheet" "~"
+			(at 157.48 99.06 0)
+			(effects
+				(font
+					(size 1.27 1.27)
+				)
+				(hide yes)
+			)
+		)
+		(property "Description" "Resistor"
+			(at 157.48 99.06 0)
+			(effects
+				(font
+					(size 1.27 1.27)
+				)
+				(hide yes)
+			)
+		)
+		(pin "2"
+		)
+		(pin "1"
+		)
+		(instances
+			(project ""
+				(path "/680d6f43-64c0-40c1-9b81-3062a08c6838"
+					(reference "R2")
+					(unit 1)
+				)

Commit message: Update schematics
Signed-off-by: LAMBS Pierre-Antoine <pierreantoine.lambs@gmail.com>
Parts:
- R2: footprint (none) -> Resistor_SMD:R_0402_1005Metric_Pad0.72x0.64mm_HandSolder
- U3: footprint QUECTEL_L96:L96 -> RF_GPS:Quectel_L96
Connections:
- net GND: now also J2.1 (Pin_1); no longer J2.2 (Pin_2)
- net VIN: now reaches C1.1, C2.1, U2.3 (VI)
- net VIN: now also J2.2 (Pin_2); no longer J2.1 (Pin_1)
Other:
- moved on the sheet: J2
Changed lines of the file:
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@@
 	)
 	(junction
-		(at 107.95 33.02)
+		(at 95.25 20.32)
 		(diameter 0)
 		(color 0 0 0 0)
@@
 	)
 	(junction
+		(at 115.57 25.4)
+		(diameter 0)
+		(color 0 0 0 0)
+	)
+	(junction
 		(at 135.89 81.28)
 		(diameter 0)
@@
 	)
 	(junction
+		(at 95.25 22.86)
+		(diameter 0)
+		(color 0 0 0 0)
+	)
+	(junction
 		(at 93.98 88.9)
 		(diameter 0)
@@
 	)
 	(junction
-		(at 93.98 81.28)
+		(at 115.57 33.02)
 		(diameter 0)
 		(color 0 0 0 0)
 	)
 	(junction
-		(at 107.95 25.4)
+		(at 93.98 81.28)
 		(diameter 0)
 		(color 0 0 0 0)
@@
 	)
 	(junction
-		(at 115.57 25.4)
-		(diameter 0)
-		(color 0 0 0 0)
-	)
-	(junction
 		(at 93.98 86.36)
 		(diameter 0)
@@
 	)
 	(junction
-		(at 115.57 33.02)
-		(diameter 0)
-		(color 0 0 0 0)
-	)
-	(junction
 		(at 135.89 66.04)
 		(diameter 0)
@@
 	(wire
 		(pts
-			(xy 101.6 30.48) (xy 107.95 30.48)
-		)
-		(stroke
-			(width 0)
-			(type default)
-		)
-	)
-	(wire
-		(pts
 			(xy 93.98 81.28) (xy 88.9 81.28)
 		)
@@
 	(wire
 		(pts
-			(xy 107.95 33.02) (xy 107.95 39.37)
-		)
-		(stroke
-			(width 0)
-			(type default)
-		)
-	)
-	(wire
-		(pts
 			(xy 134.62 71.12) (xy 139.7 71.12)
 		)
@@
 	(wire
 		(pts
+			(xy 111.76 25.4) (xy 115.57 25.4)
+		)
+		(stroke
+			(width 0)
+			(type default)
+		)
+	)
+	(wire
+		(pts
 			(xy 180.34 83.82) (xy 180.34 86.36)
 		)
@@
 	(wire
 		(pts
-			(xy 67.31 82.55) (xy 76.2 82.55)
+			(xy 95.25 20.32) (xy 97.79 20.32)
 		)
 		(stroke
@@
 	(wire
 		(pts
-			(xy 67.31 39.37) (xy 76.2 39.37)
+			(xy 67.31 82.55) (xy 76.2 82.55)
 		)
 		(stroke
@@
 	(wire
 		(pts
-			(xy 175.26 46.99) (xy 180.34 46.99)
+			(xy 67.31 39.37) (xy 76.2 39.37)
 		)
 		(stroke
@@
 	(wire
 		(pts
-			(xy 101.6 33.02) (xy 107.95 33.02)
+			(xy 175.26 46.99) (xy 180.34 46.99)
 		)
 		(stroke
@@
 	(wire
 		(pts
-			(xy 107.95 25.4) (xy 115.57 25.4)
+			(xy 93.98 66.04) (xy 96.52 66.04)
 		)
 		(stroke
@@
 	(wire
 		(pts
-			(xy 93.98 66.04) (xy 96.52 66.04)
+			(xy 180.34 78.74) (xy 185.42 78.74)
 		)
 		(stroke
@@
 	(wire
 		(pts
-			(xy 180.34 78.74) (xy 185.42 78.74)
+			(xy 135.89 58.42) (xy 135.89 60.96)
 		)
 		(stroke
@@
 	(wire
 		(pts
-			(xy 135.89 58.42) (xy 135.89 60.96)
+			(xy 90.17 93.98) (xy 96.52 93.98)
 		)
 		(stroke
@@
 	(wire
 		(pts
-			(xy 90.17 93.98) (xy 96.52 93.98)
+			(xy 111.76 33.02) (xy 115.57 33.02)
 		)
 		(stroke
@@
 	(wire
 		(pts
-			(xy 107.95 19.05) (xy 107.95 25.4)
+			(xy 88.9 72.39) (xy 88.9 76.2)
 		)
 		(stroke
@@
 	(wire
 		(pts
-			(xy 88.9 72.39) (xy 88.9 76.2)
+			(xy 156.21 25.4) (xy 163.83 25.4)
 		)
 		(stroke
@@
 	(wire
 		(pts
-			(xy 156.21 25.4) (xy 163.83 25.4)
+			(xy 38.1 125.73) (xy 43.18 125.73)
 		)
 		(stroke
@@
 	(wire
 		(pts
-			(xy 38.1 125.73) (xy 43.18 125.73)
+			(xy 93.98 22.86) (xy 95.25 22.86)
 		)
 		(stroke
@@
 	(wire
 		(pts
+			(xy 93.98 20.32) (xy 95.25 20.32)
+		)
+		(stroke
+			(width 0)
+			(type default)
+		)
+	)
+	(wire
+		(pts
 			(xy 67.31 44.45) (xy 76.2 44.45)
 		)
@@
 	(wire
 		(pts
-			(xy 107.95 30.48) (xy 107.95 25.4)
-		)
-		(stroke
-			(width 0)
-			(type default)
-		)
-	)
-	(wire
-		(pts
 			(xy 93.98 88.9) (xy 96.52 88.9)
 		)
@@
 	(wire
 		(pts
-			(xy 107.95 33.02) (xy 115.57 33.02)
+			(xy 95.25 22.86) (xy 97.79 22.86)
 		)
 		(stroke
@@
 		)
 	)
+	(label "VIN"
+		(at 111.76 25.4 180)
+		(effects
+			(font
+				(size 1.27 1.27)
+			)
+			(justify right bottom)
+		)
+	)
 	(label "STATUS_LED"
 		(at 76.2 39.37 0)
@@
 		)
 	)
+	(label "GND"
+		(at 97.79 20.32 0)
+		(effects
+			(font
+				(size 1.27 1.27)
+			)
+			(justify left bottom)
+		)
+	)
+	(label "VIN"
+		(at 97.79 22.86 0)
+		(effects
+			(font
+				(size 1.27 1.27)
+			)
+			(justify left bottom)
+		)
+	)
 	(label "ESP32_BOOT"
 		(at 76.2 34.29 0)
@@
 		)
 	)
+	(label "GND"
+		(at 111.76 33.02 180)
+		(effects
+			(font
+				(size 1.27 1.27)
+			)
+			(justify right bottom)
+		)
+	)
 	(label "DIP3"
 		(at 76.2 82.55 0)
@@
 	(symbol
 		(lib_id "power:PWR_FLAG")
-		(at 107.95 19.05 0)
+		(at 95.25 20.32 0)
 		(unit 1)
 		(exclude_from_sim no)
@@
 		(on_board yes)
 		(dnp no)
-		(fields_autoplaced yes)
 		(property "Reference" "#FLG01"
-			(at 107.95 17.145 0)
+			(at 95.25 18.415 0)
 			(effects
 				(font
@@
 		)
 		(property "Value" "PWR_FLAG"
-			(at 107.95 13.97 0)
+			(at 100.584 14.986 0)
 			(effects
 				(font
@@
 		)
 		(property "Footprint" ""
-			(at 107.95 19.05 0)
+			(at 95.25 20.32 0)
 			(effects
 				(font
@@
 		)
 		(property "Datasheet" "~"
-			(at 107.95 19.05 0)
+			(at 95.25 20.32 0)
 			(effects
 				(font
@@
 		)
 		(property "Description" "Special symbol for telling ERC where power comes from"
-			(at 107.95 19.05 0)
+			(at 95.25 20.32 0)
 			(effects
 				(font
@@
 	(symbol
 		(lib_id "Connector:Conn_01x02_Pin")
-		(at 96.52 30.48 0)
+		(at 88.9 20.32 0)
 		(unit 1)
 		(exclude_from_sim no)
@@
 		(on_board yes)
 		(dnp no)
-		(fields_autoplaced yes)
 		(property "Reference" "J2"
-			(at 97.155 25.4 0)
+			(at 89.535 15.24 0)
 			(effects
 				(font
@@
 		)
 		(property "Value" "Power Input"
-			(at 97.155 27.94 0)
+			(at 85.09 17.526 0)
 			(effects
 				(font
@@
 		)
 		(property "Footprint" "Connector_PinHeader_2.00mm:PinHeader_1x02_P2.00mm_Vertical"
-			(at 96.52 30.48 0)
+			(at 88.9 20.32 0)
 			(effects
 				(font
@@
 		)
 		(property "Datasheet" "~"
-			(at 96.52 30.48 0)
+			(at 88.9 20.32 0)
 			(effects
 				(font
@@
 		)
 		(property "Description" "Generic connector, single row, 01x02, script generated"
-			(at 96.52 30.48 0)
+			(at 88.9 20.32 0)
 			(effects
 				(font
@@
 			)
 		)
-		(property "Footprint" ""
+		(property "Footprint" "Resistor_SMD:R_0402_1005Metric_Pad0.72x0.64mm_HandSolder"
 			(at 157.48 100.838 90)
 			(effects
@@
 			)
 		)
-		(property "Footprint" "QUECTEL_L96:L96"
+		(property "Footprint" "RF_GPS:Quectel_L96"
 			(at 130.81 150.8 0)
 			(effects
@@
 	(symbol
 		(lib_id "power:PWR_FLAG")
-		(at 107.95 39.37 180)
+		(at 95.25 22.86 180)
 		(unit 1)
 		(exclude_from_sim no)
@@
 		(fields_autoplaced yes)
 		(property "Reference" "#FLG02"
-			(at 107.95 41.275 0)
+			(at 95.25 24.765 0)
 			(effects
 				(font
@@
 		)
 		(property "Value" "PWR_FLAG"
-			(at 107.95 44.45 0)
+			(at 95.25 27.94 0)
 			(effects
 				(font
@@
 		)
 		(property "Footprint" ""
-			(at 107.95 39.37 0)
+			(at 95.25 22.86 0)
 			(effects
 				(font
@@
 		)
 		(property "Datasheet" "~"
-			(at 107.95 39.37 0)
+			(at 95.25 22.86 0)
 			(effects
 				(font
@@
 		)
 		(property "Description" "Special symbol for telling ERC where power comes from"
-			(at 107.95 39.37 0)
+			(at 95.25 22.86 0)
 			(effects
 				(font

Commit message: Update schematics
Signed-off-by: LAMBS Pierre-Antoine <pierreantoine.lambs@gmail.com>
Parts:
- added TP1, TP2, TP3, TP4, TP5, TP6, TP7, TP8: TestPoint, TestPoint:TestPoint_Pad_D1.0mm, symbol Connector:TestPoint
Connections:
- net +3.3V: now also TP1.1; no longer U3.8 (V_BCKP)
- net ESP32_BOOT: now also TP6.1
- net ESP32_EN: now also TP7.1
- net GND: now also TP2.1
- net GPS_PPS: now also TP5.1
- net GPS_RX: now also TP4.1
- net GPS_TX: now also TP3.1
- net STATUS_LED: now also TP8.1
- no-connect marks 30 -> 31
Other:
- moved on the sheet: C1, C2, C3, C4, J1, R1, R2, R3, SW1, U1, U2, U3

Commit message: schematics: update schematics and add missing pull up/down
Parts:
- removed R2: 0, Resistor_SMD:R_0402_1005Metric_Pad0.72x0.64mm_HandSolder, symbol Device:R
- added C5, C6, C7: 0.1uF, Capacitor_SMD:C_0402_1005Metric_Pad0.74x0.62mm_HandSolder, symbol Device:C
- added C8: 10uF, Capacitor_SMD:C_0402_1005Metric_Pad0.74x0.62mm_HandSolder, symbol Device:C
- added TP9: TestPoint, TestPoint:TestPoint_Pad_D1.0mm, symbol Connector:TestPoint
Connections:
- net RF_OUT is gone; now on net RF_IN: U3.16 (RF_OUT)
- net +3.3V: now also C7.1, C8.1; no longer U3.23 (RESET)
- net ESP32_BOOT: now also C6.1
- net ESP32_EN: now also C5.1
- net GND: now also C5.2, C6.2, C7.2, C8.2
- net GPS_RESET: now reaches U1.30 (IO18)
- net GPS_RESET: now also U3.23 (RESET), TP9.1
- no-connect marks 31 -> 30
Other:
- moved on the sheet: R3, TP7

Commit message: schematic: update capacitor values
Signed-off-by: LAMBS Pierre-Antoine <pierreantoine.lambs@gmail.com>
Parts:
- C5, C6, C7: value 0.1uF -> 100nF
